File: blockdiagram/blockdiagram/Control_Logic.kicad_sch (KiCad schematic)
At the start: 0 parts

Commit message: updated from meeting with mateo
Changed lines of the file:
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@@
 (kicad_sch (version 20230121) (generator eeschema)
   (paper "A4")
+  (hierarchical_label "Instruction" (shape input) (at 49.53 54.61 180) (fields_autoplaced)
+    (effects (font (size 1.27 1.27)) (justify right))
+  )
   (hierarchical_label "ALU Control Signals" (shape output) (at 93.98 45.72 0) (fields_autoplaced)
     (effects (font (size 1.27 1.27)) (justify left))
