File: blockdiagram/blockdiagram/control_unit.kicad_sch (KiCad schematic)
At the start: 0 parts

Commit message: updated from meeting with mateo
Other:
- sheet Control Logic ports: added Instruction; removed none
- note added: "Add start signal when new instruction is recieved"
Changed lines of the file:
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@@
+    (stroke (width 0) (type default))
+  )
+  (wire (pts (xy 60.96 46.99) (xy 66.04 46.99))
     (stroke (width 0) (type default))
   )
@@
     (stroke (width 0) (type default))
   )
+  (wire (pts (xy 31.75 59.69) (xy 60.96 59.69))
+    (stroke (width 0) (type default))
+  )
   (wire (pts (xy 99.06 41.91) (xy 105.41 41.91))
     (stroke (width 0) (type default))
+  )
+  (wire (pts (xy 60.96 59.69) (xy 60.96 46.99))
+    (stroke (width 0) (type default))
+  )
+  (text "Add start signal when new instruction is recieved\n"
+    (at 30.48 31.75 0)
+    (effects (font (size 1.27 1.27)) (justify left bottom))
   )
   (hierarchical_label "VRF Control Signals" (shape output) (at 105.41 41.91 0) (fields_autoplaced)
@@
   (hierarchical_label "ALU Control Signals" (shape output) (at 105.41 38.1 0) (fields_autoplaced)
     (effects (font (size 1.27 1.27)) (justify left))
+  )
+  (hierarchical_label "Instruction" (shape input) (at 31.75 59.69 180) (fields_autoplaced)
+    (effects (font (size 1.27 1.27)) (justify right))
   )
   (hierarchical_label "Memory Control Signals" (shape output) (at 105.41 45.72 0) (fields_autoplaced)
@@
       (effects (font (size 1.27 1.27)) (justify left))
     )
+    (pin "Instruction" input (at 66.04 46.99 180)
+      (effects (font (size 1.27 1.27)) (justify left))
+    )
